Commit message: added python frontier exploration

File: hector_quadrotor/hector_quadrotor_description/urdf/quadrotor_velodyne.urdf.xacro (robot description, xacro)
@@ -20,4 +20,9 @@
       <origin xyz="0.05 0.0 -0.06" rpy="0 0 0"/>
     </xacro:generic_camera>
+    <!-- Backward facing camera -->
+    <xacro:include filename="$(find hector_sensors_description)/urdf/generic_camera.urdf.xacro" />
+    <xacro:generic_camera name="bottom_cam" parent="base_link" ros_topic="camera/image" cam_info_topic="camera/camera_info" update_rate="10" res_x="320" res_y="240" image_format="R8G8B8" hfov="90">
+      <origin xyz="0 0.0 -0.09" rpy="0 ${M_PI_2} 0"/>
+    </xacro:generic_camera>
     <!-- Asus Xiton Live Pro -->
     <xacro:include filename="$(find hector_sensors_description)/urdf/asus_camera.urdf.xacro" />

Commit message: removed gdb/debug from ros launch files

File: hector_quadrotor/hector_quadrotor_description/urdf/quadrotor_velodyne.urdf.xacro (robot description, xacro)
@@ -18,9 +18,9 @@
     <xacro:include filename="$(find hector_sensors_description)/urdf/generic_camera.urdf.xacro" />
     <xacro:generic_camera name="front_cam" parent="base_link" ros_topic="camera/image" cam_info_topic="camera/camera_info" update_rate="10" res_x="320" res_y="240" image_format="R8G8B8" hfov="90">
-      <origin xyz="0.05 0.0 -0.06" rpy="0 0 0"/>
+      <origin xyz="0.05 0.0 -0.06" rpy="0 0.43 0"/>
     </xacro:generic_camera>
     <!-- Backward facing camera -->
     <xacro:include filename="$(find hector_sensors_description)/urdf/generic_camera.urdf.xacro" />
-    <xacro:generic_camera name="bottom_cam" parent="base_link" ros_topic="camera/image" cam_info_topic="camera/camera_info" update_rate="10" res_x="320" res_y="240" image_format="R8G8B8" hfov="90">
+    <xacro:generic_camera name="bottom_cam" parent="base_link" ros_topic="camera/image" cam_info_topic="camera/camera_info" update_rate="10" res_x="512" res_y="512" image_format="R8G8B8" hfov="90">
       <origin xyz="0 0.0 -0.09" rpy="0 ${M_PI_2} 0"/>
     </xacro:generic_camera>

Commit message: added new lidar on top/not sure if it helps though

File: hector_quadrotor/hector_quadrotor_description/urdf/quadrotor_velodyne.urdf.xacro (robot description, xacro)
@@ -14,4 +14,12 @@
     	<!-- Forward facing rotation -->
     	<origin xyz="0.0 0.0 -0.097" rpy="${M_PI_2} 0 0"/>
+    </xacro:vlp16>
+    <!-- VLP-16 mounted above the quadrotor body -->
+    <xacro:include filename="$(find hector_sensors_description)/urdf/vlp16.urdf.xacro" />
+    <xacro:vlp16 name="laser1" parent="base_link" ros_topic="velodyne_points1">
+      <!-- Sideways facing rotation -->
+      <!--<origin xyz="0.0 0.0 -0.097" rpy="${M_PI_2} 0 ${M_PI_2}"/>-->
+      <!-- Forward facing rotation -->
+      <origin xyz="0.0 0.0 0.097" rpy="${M_PI_2} ${M_PI} 0"/>
     </xacro:vlp16>
     <!-- Forward facing camera -->

Commit message: creating new world/need to finish rotation and adding one more bridge model

File: hector_quadrotor/hector_quadrotor_description/urdf/quadrotor_velodyne.urdf.xacro (robot description, xacro)
@@ -14,12 +14,4 @@
     	<!-- Forward facing rotation -->
     	<origin xyz="0.0 0.0 -0.097" rpy="${M_PI_2} 0 0"/>
-    </xacro:vlp16>
-    <!-- VLP-16 mounted above the quadrotor body -->
-    <xacro:include filename="$(find hector_sensors_description)/urdf/vlp16.urdf.xacro" />
-    <xacro:vlp16 name="laser1" parent="base_link" ros_topic="velodyne_points1">
-      <!-- Sideways facing rotation -->
-      <!--<origin xyz="0.0 0.0 -0.097" rpy="${M_PI_2} 0 ${M_PI_2}"/>-->
-      <!-- Forward facing rotation -->
-      <origin xyz="0.0 0.0 0.097" rpy="${M_PI_2} ${M_PI} 0"/>
     </xacro:vlp16>
     <!-- Forward facing camera -->
